File: I2C-port-expander.kicad_pcb (KiCad board)
At the start: 2 copper layers, 100 x 100 mm, 16 parts, among them J1 Conn_01x05, J2 Conn_01x08, J3 Conn_01x08, U1 PCF8575C

Commit message: update,
Parts:
- added D1: LED_GREEN, LED_SMD:LED_0805_2012Metric_Castellated, F.Cu at (14.4, 27.9)
- added R4: R511, Resistor_SMD:R_0805_2012Metric_Pad1.15x1.40mm_HandSolder, F.Cu at (17.4, 27.8)
- moved C2 11.2 mm to (26.7, 21.3), turned to 90 degrees
- moved J1 10.1 mm to (10.0, 27.5), turned to 180 degrees
- moved C1 9.91 mm to (23.7, 21.3), turned to 90 degrees
- moved R1 7.23 mm to (20.5, 21.4), turned to 90 degrees
- moved U1 6.83 mm to (36.5, 28.1)
- moved JP3 6.69 mm to (28.0, 27.8), turned to 270 degrees
- moved JP1 5.99 mm to (21.0, 27.9), turned to 270 degrees
- moved JP2 3.41 mm to (24.5, 27.9), turned to 270 degrees
- moved R2 3.41 mm to (18.2, 21.4), turned to 90 degrees
- moved J3 1.20 mm to (41.8, 16.2)
- moved R3 0.44 mm to (15.8, 21.4), turned to 90 degrees
Connections:
- J1 pad 2: Net-(J1-Pad2) -> +3V3
- J1 pad 3: Net-(J1-Pad3) -> /INT
- J1 pad 4: Net-(J1-Pad4) -> /SCL
- J1 pad 5: +3V3 -> /SDA
- R1 pad 2: Net-(J1-Pad4) -> /SDA
- R2 pad 2: Net-(J1-Pad3) -> /SCL
- R3 pad 2: Net-(J1-Pad2) -> /INT
Routing:
- net +3V3: track 0.00 -> 48.3 mm
- net /SCL: track 0.00 -> 42.6 mm, vias 0 -> 1
- net /SDA: track 0.00 -> 41.5 mm, vias 0 -> 1
- net /INT: track 0.00 -> 39.7 mm, vias 0 -> 1
- net /PO0: track 0.00 -> 29.3 mm, vias 0 -> 1
- net /A0: track 0.00 -> 26.9 mm, vias 0 -> 2
- net GND: track 0.00 -> 26.3 mm
- net /PO2: track 0.00 -> 25.9 mm, vias 0 -> 1
- net /PO1: track 0.00 -> 25.8 mm, vias 0 -> 1
- net /PO7: track 0.00 -> 24.7 mm, vias 0 -> 1
- net /PO3: track 0.00 -> 23.8 mm, vias 0 -> 1
- net /PO5: track 0.00 -> 23.4 mm, vias 0 -> 1
- net /PO4: track 0.00 -> 23.0 mm, vias 0 -> 1
- net /PO6: track 0.00 -> 22.9 mm, vias 0 -> 1
- net /P17: track 0.00 -> 17.0 mm, vias 0 -> 1
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- added copper zone on B.Cu, net GND
- added copper zone on F.Cu, net GND
Other:
- net class 3V3 added: clearance 0.2, trace_width 0.5, via_dia 0.8, via_drill 0.4
- net class GND added: clearance 0.2, trace_width 0.75, via_dia 0.8, via_drill 0.4

Commit message: update,
Parts:
- moved R1 0.76 mm to (21.2, 21.3)
- moved R2 0.34 mm to (18.5, 21.3)
- moved C1 0.28 mm to (24.0, 21.3)
- moved R3 0.10 mm to (15.8, 21.3)
Routing:
- net /SDA: track 41.5 -> 51.3 mm
- net /A0: track 26.9 -> 17.8 mm
- net /P17: track 17.0 -> 18.8 mm
- net /SCL: track 42.6 -> 44.4 mm
- net /PO0: track 29.3 -> 28.1 mm
- net /A1: track 13.1 -> 14.1 mm
- net /PO7: track 24.7 -> 23.9 mm
- net /INT: track 39.7 -> 38.9 mm
- net +3V3: track 48.3 -> 47.6 mm
- net /PO2: track 25.9 -> 25.3 mm
- net GND: vias 0 -> 9
Other:
- board size 100 x 100 mm -> 50 x 35 mm
