File: I2C-port-expander.kicad_pcb (KiCad board)
At the start: 2 copper layers, 50 x 35 mm, 18 parts, among them J1 Conn_01x05, J2 Conn_01x08, J3 Conn_01x08, U1 PCF8575C

Commit message: update jumper marking,
Other:
- board text added: "I2C PORT EXPANDER"
Changed lines of the file:
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@@
   (general
     (thickness 1.6)
-    (drawings 12)
+    (drawings 13)
     (tracks 279)
     (zones 0)
@@
       (effects (font (size 1 1) (thickness 0.15)))
     )
-    (fp_text user 3 (at 2.6 0 270) (layer F.SilkS)
-      (effects (font (size 1 1) (thickness 0.15)))
-    )
-    (fp_text user 1 (at -2.6 0 270) (layer F.SilkS)
+    (fp_text user G (at 2.6 0 270) (layer F.SilkS)
+      (effects (font (size 1 1) (thickness 0.15)))
+    )
+    (fp_text user + (at -2.6 0 270) (layer F.SilkS)
       (effects (font (size 1 1) (thickness 0.15)))
     )
@@
     (fp_line (start 1.4 1) (end -1.4 1) (layer F.SilkS) (width 0.12))
     (fp_line (start -2.05 0.3) (end -2.05 -0.3) (layer F.SilkS) (width 0.12))
-    (fp_text user 1 (at -2.6 0 270) (layer F.SilkS)
-      (effects (font (size 1 1) (thickness 0.15)))
-    )
-    (fp_text user 3 (at 2.6 0 270) (layer F.SilkS)
+    (fp_text user + (at -2.6 0 270) (layer F.SilkS)
+      (effects (font (size 1 1) (thickness 0.15)))
+    )
+    (fp_text user G (at 2.6 0 270) (layer F.SilkS)
       (effects (font (size 1 1) (thickness 0.15)))
     )
@@
       (effects (font (size 1 1) (thickness 0.15)))
     )
-    (fp_text user 3 (at 2.6 0 270) (layer F.SilkS)
-      (effects (font (size 1 1) (thickness 0.15)))
-    )
-    (fp_text user 1 (at -2.6 0 270) (layer F.SilkS)
+    (fp_text user G (at 2.6 0 270) (layer F.SilkS)
+      (effects (font (size 1 1) (thickness 0.15)))
+    )
+    (fp_text user + (at -2.6 0 270) (layer F.SilkS)
       (effects (font (size 1 1) (thickness 0.15)))
     )
@@
     )
   )
+  (gr_text "I2C PORT EXPANDER" (at 30 35) (layer B.SilkS)
+    (effects (font (size 2 2) (thickness 0.3)) (justify mirror))
+  )
   (gr_line (start 10 40) (end 50 40) (layer Edge.Cuts) (width 0.15))
