File: I2C-port-expander.kicad_pcb (KiCad board)
At the start: 2 copper layers, 50 x 35 mm, 18 parts, among them J1 Conn_01x05, J2 Conn_01x08, J3 Conn_01x08, U1 PCF8575C

Commit message: update,
Parts:
- J1: footprint Connector_PinHeader_2.54mm:PinHeader_1x05_P2.54mm_Vertical -> footprint-lib.pretty:Pin_Header_Straight_1x05_Pitch2.54mm
- J2, J3: footprint Connector_PinHeader_2.54mm:PinHeader_1x08_P2.54mm_Vertical -> footprint-lib.pretty:Pin_Header_Straight_1x08_Pitch2.54mm
- moved JP3 0.20 mm to (28.0, 27.9)
Routing:
- net /P14: track 12.0 -> 15.0 mm
- net /P16: track 15.3 -> 17.8 mm
- net /P12: track 9.12 -> 11.3 mm
- net /P11: track 8.57 -> 10.6 mm
- net +3V3: track 47.6 -> 45.6 mm
- net /SCL: track 44.4 -> 46.2 mm
- net /PO3: track 23.7 -> 24.7 mm
- net /PO0: track 28.1 -> 29.0 mm
- net /P13: track 10.4 -> 11.2 mm
- net /PO5: track 23.4 -> 22.7 mm
- net /PO1: track 25.9 -> 26.5 mm
- net GND: track 26.3 -> 26.0 mm, vias 9 -> 14
Other:
- net class 3V3: trace_width 0.5 -> 0.75; via_dia 0.8 -> 1.2
- net class GND: trace_width 0.75 -> 1; via_dia 0.8 -> 1.5

Commit message: update,
Routing:
- net /PO4: vias 1 -> 2
- net GND: vias 14 -> 22
- net /PO7: vias 1 -> 2
- net /PO6: vias 1 -> 3
Changed lines of the file:
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@@
     (thickness 1.6)
     (drawings 13)
-    (tracks 297)
+    (tracks 313)
     (zones 0)
     (modules 18)
@@
   (segment (start 34.38 10) (end 34.38 11.98) (width 0.25) (layer B.Cu) (net 9))
   (segment (start 37.25 28.275) (end 37.25 27.5) (width 0.25) (layer F.Cu) (net 9))
-  (segment (start 35.4 13) (end 35.4 19.1) (width 0.25) (layer B.Cu) (net 9))
+  (segment (start 35.4 13) (end 35.4 13.3858) (width 0.25) (layer B.Cu) (net 9))
   (segment (start 34.38 11.98) (end 35.4 13) (width 0.25) (layer B.Cu) (net 9))
+  (segment (start 35.4 13.3858) (end 35.4 19.1) (width 0.25) (layer B.Cu) (net 9))
+  (via (at 35.4 13.3858) (size 0.8) (drill 0.4) (layers F.Cu B.Cu) (net 9))
   (segment (start 36.92 10) (end 36.92 11.02) (width 0.25) (layer B.Cu) (net 10) (status 10))
   (segment (start 36.92 11.02) (end 38 12.1) (width 0.25) (layer B.Cu) (net 10))
@@
   (segment (start 39.5 22.4) (end 40.6 21.3) (width 0.25) (layer B.Cu) (net 11))
   (segment (start 38.75 31.675) (end 38.75 29) (width 0.25) (layer F.Cu) (net 11) (status 10))
-  (segment (start 40.6 21.3) (end 40.6 13.4) (width 0.25) (layer B.Cu) (net 11))
+  (segment (start 40.6 21.3) (end 40.6 19.5707) (width 0.25) (layer B.Cu) (net 11))
   (via (at 39.5 27) (size 0.8) (drill 0.4) (layers F.Cu B.Cu) (net 11))
   (segment (start 40.6 13.4) (end 39.46 12.26) (width 0.25) (layer B.Cu) (net 11))
@@
   (segment (start 39.5 28.25) (end 39.5 27) (width 0.25) (layer F.Cu) (net 11))
   (segment (start 39.46 12.26) (end 39.46 10) (width 0.25) (layer B.Cu) (net 11) (status 20))
+  (segment (start 40.6 13.4) (end 40.6 13.4) (width 0.25) (layer B.Cu) (net 11))
+  (via (at 40.6 13.4) (size 0.8) (drill 0.4) (layers F.Cu B.Cu) (net 11))
+  (segment (start 40.6 19.5707) (end 40.6 13.4) (width 0.25) (layer B.Cu) (net 11))
+  (via (at 40.6 19.5707) (size 0.8) (drill 0.4) (layers F.Cu B.Cu) (net 11))
   (via (at 41.7 27.8) (size 0.8) (drill 0.4) (layers F.Cu B.Cu) (net 12))
   (segment (start 39.4 31.675) (end 39.4 30.1) (width 0.25) (layer F.Cu) (net 12))
   (segment (start 42 13.6) (end 42 10) (width 0.25) (layer B.Cu) (net 12) (status 20))
   (segment (start 39.4 30.1) (end 41.7 27.8) (width 0.25) (layer F.Cu) (net 12))
-  (segment (start 41.7 27.8) (end 41.7 22.55) (width 0.25) (layer B.Cu) (net 12))
+  (segment (start 41.7 27.8) (end 41.7 24.5999) (width 0.25) (layer B.Cu) (net 12))
   (segment (start 43.4 20.85) (end 43.4 15) (width 0.25) (layer B.Cu) (net 12))
   (segment (start 41.7 22.55) (end 43.4 20.85) (width 0.25) (layer B.Cu) (net 12))
   (segment (start 43.4 15) (end 42 13.6) (width 0.25) (layer B.Cu) (net 12))
+  (segment (start 41.7 24.5999) (end 41.7 22.55) (width 0.25) (layer B.Cu) (net 12))
+  (via (at 41.7 24.5999) (size 0.8) (drill 0.4) (layers F.Cu B.Cu) (net 12))
   (segment (start 23.7 20.25) (end 26.7 20.25) (width 1) (layer F.Cu) (net 13))
   (segment (start 21 29.25) (end 24.5 29.25) (width 1) (layer F.Cu) (net 13))
@@
   (segment (start 10 27.5) (end 11.467499 27.5) (width 1) (layer F.Cu) (net 13))
   (via (at 19.5326 16.9418) (size 1.5) (drill 0.4) (layers F.Cu B.Cu) (net 13))
-  (via (at 16.1798 24.0792) (size 1.5) (drill 0.4) (layers F.Cu B.Cu) (net 13))
-  (via (at 14.097 18.4658) (size 1.5) (drill 0.4) (layers F.Cu B.Cu) (net 13))
+  (via (at 16.1798 24.0792) (size 1) (drill 0.4) (layers F.Cu B.Cu) (net 13))
+  (via (at 14.0589 18.7706) (size 1.5) (drill 0.4) (layers F.Cu B.Cu) (net 13))
   (via (at 13.7668 21.5392) (size 0.8) (drill 0.4) (layers F.Cu B.Cu) (net 13))
-  (via (at 12.7 23.5966) (size 1.5) (drill 0.4) (layers F.Cu B.Cu) (net 13))
+  (via (at 12.7 23.5966) (size 0.8) (drill 0.4) (layers F.Cu B.Cu) (net 13))
   (via (at 7.0612 21.2344) (size 1.5) (drill 0.4) (layers F.Cu B.Cu) (net 13))
   (via (at 30.9626 28.8036) (size 0.8) (drill 0.4) (layers F.Cu B.Cu) (net 13))
   (via (at 30.3 25.9) (size 0.8) (drill 0.4) (layers F.Cu B.Cu) (net 13))
-  (via (at 21.6662 24.2062) (size 1.5) (drill 0.4) (layers F.Cu B.Cu) (net 13))
-  (via (at 44.2722 21.2344) (size 1.5) (drill 0.4) (layers F.Cu B.Cu) (net 13))
+  (via (at 21.6662 24.2062) (size 1) (drill 0.4) (layers F.Cu B.Cu) (net 13))
+  (via (at 46.9646 21.5392) (size 1.5) (drill 0.4) (layers F.Cu B.Cu) (net 13))
   (via (at 47.1932 28.1178) (size 1.5) (drill 0.4) (layers F.Cu B.Cu) (net 13))
   (via (at 17.9324 8.2804) (size 1.5) (drill 0.4) (layers F.Cu B.Cu) (net 13))
   (via (at 15.4686 36.5506) (size 1.5) (drill 0.4) (layers F.Cu B.Cu) (net 13))
-  (via (at 40.4114 37.6428) (size 1.5) (drill 0.4) (layers F.Cu B.Cu) (net 13))
+  (via (at 40.6527 36.0299) (size 1.5) (drill 0.4) (layers F.Cu B.Cu) (net 13))
+  (via (at 24.9428 24.6126) (size 0.8) (drill 0.4) (layers F.Cu B.Cu) (net 13))
+  (via (at 27.432 23.9268) (size 0.8) (drill 0.4) (layers F.Cu B.Cu) (net 13))
+  (via (at 23.4061 31.877) (size 1.5) (drill 0.4) (layers F.Cu B.Cu) (net 13))
+  (via (at 31.5341 13.1572) (size 1.5) (drill 0.4) (layers F.Cu B.Cu) (net 13))
+  (via (at 25.5778 13.1699) (size 0.8) (drill 0.4) (layers F.Cu B.Cu) (net 13))
+  (via (at 22.7711 18.4023) (size 0.8) (drill 0.4) (layers F.Cu B.Cu) (net 13))
+  (via (at 12.3952 26.9875) (size 0.8) (drill 0.4) (layers F.Cu B.Cu) (net 13))
+  (via (at 41.6814 30.2514) (size 0.8) (drill 0.4) (layers F.Cu B.Cu) (net 13))
   (via (at 41.75 20.5) (size 0.8) (drill 0.4) (layers F.Cu B.Cu) (net 14))
   (segment (start 41.8 20.45) (end 41.75 20.5) (width 0.25) (layer B.Cu) (net 14))
@@
     (connect_pads (clearance 0.508))
     (min_thickness 0.254)
-    (fill yes (arc_segments 16) (thermal_gap 0.508) (thermal_bridge_width 0.508))
+    (fill (arc_segments 16) (thermal_gap 0.508) (thermal_bridge_width 0.508))
     (polygon
       (pts
@@
     (connect_pads (clearance 0.508))
     (min_thickness 0.254)
-    (fill yes (arc_segments 16) (thermal_gap 0.508) (thermal_bridge_width 0.508))
+    (fill (arc_segments 16) (thermal_gap 0.508) (thermal_bridge_width 0.508))
     (polygon
       (pts
