File: I2C-port-expander.sch (KiCad schematic (older format))
At the start: 12 parts, among them J1 Conn_01x05, J2 Conn_01x08, J3 Conn_01x08, U1 PCF8575C

Commit message: update,
Parts:
- added D?: LED_GREEN, symbol taobao-components:LED_GREEN
- added R?: R511, symbol taobao-r:R511
- C1, C2: renamed from C?; footprint (none) -> Capacitor_SMD:C_0805_2012Metric_Pad1.15x1.40mm_HandSolder
Connections:
- net +3V3: now also J1.2 (Pin_2), R?.1; no longer J1.5 (Pin_5)
- net GND: now also D?.1 (K)
- net INT: now also J1.3 (Pin_3), R3.2
- net SCL: now also J1.4 (Pin_4), R2.2
- net SDA: now also J1.5 (Pin_5), R1.2
- new net: D?.2 (A), R?.2
Other:
- moved on the sheet: R1, R2, R3
Changed lines of the file:
@@
 F 3 "~" H 5450 2400 50  0001 C CNN
 	1    5450 2400
-	-1   0    0    1
+	-1   0    0    -1
 $EndComp
 $Comp
 L power:GND #PWR0109
 U 1 1 5BC7D515
-P 5800 2700
-F 0 "#PWR0109" H 5800 2450 50  0001 C CNN
-F 1 "GND" H 5850 2500 50  0000 C CNN
-F 2 "" H 5800 2700 50  0001 C CNN
-F 3 "" H 5800 2700 50  0001 C CNN
-	1    5800 2700
-	1    0    0    -1
-$EndComp
-Wire Wire Line
-	5800 2700 5800 2600
-Wire Wire Line
-	5800 2600 5650 2600
+P 5800 2100
+F 0 "#PWR0109" H 5800 1850 50  0001 C CNN
+F 1 "GND" H 5850 1900 50  0000 C CNN
+F 2 "" H 5800 2100 50  0001 C CNN
+F 3 "" H 5800 2100 50  0001 C CNN
+	1    5800 2100
+	1    0    0    1
+$EndComp
+Wire Wire Line
+	5800 2100 5800 2200
+Wire Wire Line
+	5800 2200 5650 2200
 $Comp
 L taobao-r:R472 R1
 U 1 1 5BC7DDB9
-P 6100 2300
-F 0 "R1" V 5850 2300 50  0000 C CNN
-F 1 "R472" V 5950 2300 50  0000 C CNN
-F 2 "Resistor_SMD:R_0805_2012Metric_Pad1.15x1.40mm_HandSolder" H 6100 2300 50  0001 C CNN
-F 3 "~" H 6100 2300 50  0001 C CNN
-	1    6100 2300
-	0    1    1    0
+P 6100 2600
+F 0 "R1" V 5850 2600 50  0000 C CNN
+F 1 "R472" V 5950 2600 50  0000 C CNN
+F 2 "Resistor_SMD:R_0805_2012Metric_Pad1.15x1.40mm_HandSolder" H 6100 2600 50  0001 C CNN
+F 3 "~" H 6100 2600 50  0001 C CNN
+	1    6100 2600
+	0    1    -1   0
 $EndComp
 $Comp
 L taobao-r:R472 R2
 U 1 1 5BC7DDE8
+P 6100 2500
+F 0 "R2" V 5850 2500 50  0000 C CNN
+F 1 "R472" V 5950 2500 50  0000 C CNN
+F 2 "Resistor_SMD:R_0805_2012Metric_Pad1.15x1.40mm_HandSolder" H 6100 2500 50  0001 C CNN
+F 3 "~" H 6100 2500 50  0001 C CNN
+	1    6100 2500
+	0    1    -1   0
+$EndComp
+$Comp
+L customized_power:+3V3 #PWR0110
+U 1 1 5BC7DE60
+P 6050 2100
+F 0 "#PWR0110" H 6050 1950 50  0001 C CNN
+F 1 "+3V3" H 6050 2300 50  0000 C CNN
+F 2 "" H 6050 2100 50  0001 C CNN
+F 3 "" H 6050 2100 50  0001 C CNN
+	1    6050 2100
+	-1   0    0    -1
+$EndComp
+$Comp
+L taobao-r:R472 R3
+U 1 1 5BC7E71E
 P 6100 2400
-F 0 "R2" V 5850 2400 50  0000 C CNN
+F 0 "R3" V 5850 2400 50  0000 C CNN
 F 1 "R472" V 5950 2400 50  0000 C CNN
 F 2 "Resistor_SMD:R_0805_2012Metric_Pad1.15x1.40mm_HandSolder" H 6100 2400 50  0001 C CNN
 F 3 "~" H 6100 2400 50  0001 C CNN
 	1    6100 2400
-	0    1    1    0
-$EndComp
-$Comp
-L customized_power:+3V3 #PWR0110
-U 1 1 5BC7DE60
-P 5800 2100
-F 0 "#PWR0110" H 5800 1950 50  0001 C CNN
-F 1 "+3V3" H 5850 2300 50  0000 C CNN
-F 2 "" H 5800 2100 50  0001 C CNN
-F 3 "" H 5800 2100 50  0001 C CNN
-	1    5800 2100
-	1    0    0    -1
-$EndComp
-Wire Wire Line
-	5800 2100 5800 2200
-Wire Wire Line
-	5800 2200 5650 2200
-$Comp
-L taobao-r:R472 R3
-U 1 1 5BC7E71E
-P 6100 2500
-F 0 "R3" V 5850 2500 50  0000 C CNN
-F 1 "R472" V 5950 2500 50  0000 C CNN
-F 2 "Resistor_SMD:R_0805_2012Metric_Pad1.15x1.40mm_HandSolder" H 6100 2500 50  0001 C CNN
-F 3 "~" H 6100 2500 50  0001 C CNN
-	1    6100 2500
-	0    1    1    0
-$EndComp
-$Comp
-L customized_power:+3V3 #PWR0111
-U 1 1 5BC7E73E
-P 6450 2100
-F 0 "#PWR0111" H 6450 1950 50  0001 C CNN
-F 1 "+3V3" H 6500 2300 50  0000 C CNN
-F 2 "" H 6450 2100 50  0001 C CNN
-F 3 "" H 6450 2100 50  0001 C CNN
-	1    6450 2100
-	1    0    0    -1
-$EndComp
-Wire Wire Line
-	6450 2100 6450 2300
-Wire Wire Line
-	6450 2300 6200 2300
+	0    1    -1   0
+$EndComp
+Wire Wire Line
+	6450 2600 6200 2600
+Wire Wire Line
+	6200 2500 6450 2500
+Wire Wire Line
+	6450 2500 6450 2600
 Wire Wire Line
 	6200 2400 6450 2400
 Wire Wire Line
-	6450 2400 6450 2300
-Connection ~ 6450 2300
-Wire Wire Line
-	6200 2500 6450 2500
-Wire Wire Line
-	6450 2500 6450 2400
-Connection ~ 6450 2400
-Wire Wire Line
-	5650 2300 6000 2300
+	6450 2400 6450 2500
+Connection ~ 6450 2500
+Wire Wire Line
+	5650 2600 6000 2600
+Wire Wire Line
+	5650 2500 6000 2500
 Wire Wire Line
 	5650 2400 6000 2400
-Wire Wire Line
-	5650 2500 6000 2500
 $Comp
 L Connector_Generic:Conn_01x08 J2
@@
 P17
 $Comp
-L customized_power:+3V3 #PWR?
+L customized_power:+3V3 #PWR0112
 U 1 1 5BC8E801
 P 8150 1700
-F 0 "#PWR?" H 8150 1550 50  0001 C CNN
+F 0 "#PWR0112" H 8150 1550 50  0001 C CNN
 F 1 "+3V3" H 8200 1900 50  0000 C CNN
 F 2 "" H 8150 1700 50  0001 C CNN
@@
 $EndComp
 $Comp
-L power:GND #PWR?
+L power:GND #PWR0113
 U 1 1 5BC8E852
 P 8150 2300
-F 0 "#PWR?" H 8150 2050 50  0001 C CNN
+F 0 "#PWR0113" H 8150 2050 50  0001 C CNN
 F 1 "GND" H 8200 2100 50  0000 C CNN
 F 2 "" H 8150 2300 50  0001 C CNN
@@
 $EndComp
 $Comp
-L taobao-c:C106 C?
+L taobao-c:C106 C1
 U 1 1 5BC8E8F3
 P 8150 1950
-F 0 "C?" H 8250 2000 50  0000 L CNN
+F 0 "C1" H 8250 2000 50  0000 L CNN
 F 1 "C106" H 8250 1950 50  0000 L CNN
-F 2 "" H 8150 1950 50  0001 C CNN
+F 2 "Capacitor_SMD:C_0805_2012Metric_Pad1.15x1.40mm_HandSolder" H 8150 1950 50  0001 C CNN
 F 3 "~" H 8150 1950 50  0001 C CNN
 	1    8150 1950
@@
 	8150 2050 8150 2300
 $Comp
-L customized_power:+3V3 #PWR?
+L customized_power:+3V3 #PWR0114
 U 1 1 5BC913F6
 P 8650 1700
-F 0 "#PWR?" H 8650 1550 50  0001 C CNN
+F 0 "#PWR0114" H 8650 1550 50  0001 C CNN
 F 1 "+3V3" H 8700 1900 50  0000 C CNN
 F 2 "" H 8650 1700 50  0001 C CNN
@@
 $EndComp
 $Comp
-L power:GND #PWR?
+L power:GND #PWR0115
 U 1 1 5BC91417
 P 8650 2300
-F 0 "#PWR?" H 8650 2050 50  0001 C CNN
+F 0 "#PWR0115" H 8650 2050 50  0001 C CNN
 F 1 "GND" H 8700 2100 50  0000 C CNN
 F 2 "" H 8650 2300 50  0001 C CNN
@@
 $EndComp
 $Comp
-L taobao-c:C104 C?
+L taobao-c:C104 C2
 U 1 1 5BC914A7
 P 8650 1950
-F 0 "C?" H 8750 2000 50  0000 L CNN
+F 0 "C2" H 8750 2000 50  0000 L CNN
 F 1 "C104" H 8750 1950 50  0000 L CNN
-F 2 "" H 8650 1950 50  0001 C CNN
+F 2 "Capacitor_SMD:C_0805_2012Metric_Pad1.15x1.40mm_HandSolder" H 8650 1950 50  0001 C CNN
 F 3 "~" H 8650 1950 50  0001 C CNN
 	1    8650 1950
@@
 Wire Wire Line
 	8650 2050 8650 2300
+Text Label 5700 2600 0    50   ~ 0
+SDA
+Text Label 5700 2500 0    50   ~ 0
+SCL
+Text Label 5700 2400 0    50   ~ 0
+INT
+Wire Wire Line
+	5650 2300 6050 2300
+Wire Wire Line
+	6050 2300 6050 2100
+$Comp
+L customized_power:+3V3 #PWR0111
+U 1 1 5BC97E54
+P 6450 2100
+F 0 "#PWR0111" H 6450 1950 50  0001 C CNN
+F 1 "+3V3" H 6450 2300 50  0000 C CNN
+F 2 "" H 6450 2100 50  0001 C CNN
+F 3 "" H 6450 2100 50  0001 C CNN
+	1    6450 2100
+	-1   0    0    -1
+$EndComp
+Wire Wire Line
+	6450 2400 6450 2100
+Connection ~ 6450 2400
+$Comp
+L customized_power:+3V3 #PWR?
+U 1 1 5BC9B31F
+P 9400 1700
+F 0 "#PWR?" H 9400 1550 50  0001 C CNN
+F 1 "+3V3" H 9450 1900 50  0000 C CNN
+F 2 "" H 9400 1700 50  0001 C CNN
+F 3 "" H 9400 1700 50  0001 C CNN
+	1    9400 1700
+	1    0    0    -1
+$EndComp
+$Comp
+L taobao-r:R511 R?
+U 1 1 5BC9B642
+P 9400 1950
+F 0 "R?" H 9500 2000 50  0000 L CNN
+F 1 "R511" H 9500 1950 50  0000 L CNN
+F 2 "" H 9400 1950 50  0001 C CNN
+F 3 "~" H 9400 1950 50  0001 C CNN
+	1    9400 1950
+	1    0    0    -1
+$EndComp
+$Comp
+L taobao-components:LED_GREEN D?
+U 1 1 5BC9B79A
+P 9400 2250
+F 0 "D?" V 9450 2150 50  0000 R CNN
+F 1 "LED_GREEN" V 9400 2150 50  0000 R CNN
+F 2 "" V 9400 2250 50  0001 C CNN
+F 3 "~" V 9400 2250 50  0001 C CNN
+	1    9400 2250
+	0    -1   -1   0
+$EndComp
+$Comp
+L power:GND #PWR?
+U 1 1 5BC9B899
+P 9400 2450
+F 0 "#PWR?" H 9400 2200 50  0001 C CNN
+F 1 "GND" H 9450 2250 50  0000 C CNN
+F 2 "" H 9400 2450 50  0001 C CNN
+F 3 "" H 9400 2450 50  0001 C CNN
+	1    9400 2450
+	1    0    0    -1
+$EndComp
+Wire Wire Line
+	9400 1700 9400 1850
+Wire Wire Line
+	9400 2050 9400 2150
+Wire Wire Line
+	9400 2350 9400 2450
 $EndSCHEMATC

Commit message: update,
Parts:
- D1: renamed from D?; footprint (none) -> LED_SMD:LED_0805_2012Metric_Castellated
- R4: renamed from R?; footprint (none) -> Resistor_SMD:R_0805_2012Metric_Pad1.15x1.40mm_HandSolder
Changed lines of the file:
@@
 Connection ~ 6450 2400
 $Comp
-L customized_power:+3V3 #PWR?
+L customized_power:+3V3 #PWR0116
 U 1 1 5BC9B31F
 P 9400 1700
-F 0 "#PWR?" H 9400 1550 50  0001 C CNN
+F 0 "#PWR0116" H 9400 1550 50  0001 C CNN
 F 1 "+3V3" H 9450 1900 50  0000 C CNN
 F 2 "" H 9400 1700 50  0001 C CNN
@@
 $EndComp
 $Comp
-L taobao-r:R511 R?
+L taobao-r:R511 R4
 U 1 1 5BC9B642
 P 9400 1950
-F 0 "R?" H 9500 2000 50  0000 L CNN
+F 0 "R4" H 9500 2000 50  0000 L CNN
 F 1 "R511" H 9500 1950 50  0000 L CNN
-F 2 "" H 9400 1950 50  0001 C CNN
+F 2 "Resistor_SMD:R_0805_2012Metric_Pad1.15x1.40mm_HandSolder" H 9400 1950 50  0001 C CNN
 F 3 "~" H 9400 1950 50  0001 C CNN
 	1    9400 1950
@@
 $EndComp
 $Comp
-L taobao-components:LED_GREEN D?
+L taobao-components:LED_GREEN D1
 U 1 1 5BC9B79A
 P 9400 2250
-F 0 "D?" V 9450 2150 50  0000 R CNN
+F 0 "D1" V 9450 2150 50  0000 R CNN
 F 1 "LED_GREEN" V 9400 2150 50  0000 R CNN
-F 2 "" V 9400 2250 50  0001 C CNN
+F 2 "LED_SMD:LED_0805_2012Metric_Castellated" V 9400 2250 50  0001 C CNN
 F 3 "~" V 9400 2250 50  0001 C CNN
 	1    9400 2250
@@
 $EndComp
 $Comp
-L power:GND #PWR?
+L power:GND #PWR0117
 U 1 1 5BC9B899
 P 9400 2450
-F 0 "#PWR?" H 9400 2200 50  0001 C CNN
+F 0 "#PWR0117" H 9400 2200 50  0001 C CNN
 F 1 "GND" H 9450 2250 50  0000 C CNN
 F 2 "" H 9400 2450 50  0001 C CNN
